File: UGR/New_Screen_26/UGR_Driver_Screen_26_PCB/UGR_Driver_Screen_26.kicad_sch (KiCad schematic)
At the start: 54 parts, among them J2 USB_B_Micro, J3 Conn_02x20_Socket, J4 Conn_01x06, U1 TPS562200, U2 STM32F767VGTx, U3 SI2347DS-T1-GE3, U4 MCP2562-E-MF, U5 SI2347DS-T1-GE3, U6 SI2347DS-T1-GE3, U7 SI2347DS-T1-GE3, U8 SI2347DS-T1-GE3, U9 SI2347DS-T1-GE3

Commit message: Updates
Other:
- note added: "NOTE: SCHEMATIC PINS ARE IN THE WRONG ORDER BUT THE FOOTPRINT PINS ARE IN THE RIGHT ORDER"
Changed lines of the file:
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@@
+		)
+	)
+	(text "NOTE: SCHEMATIC PINS ARE IN THE WRONG ORDER BUT THE FOOTPRINT PINS ARE IN THE RIGHT ORDER\n"
+		(exclude_from_sim no)
+		(at 321.056 108.458 0)
+		(effects
+			(font
+				(size 1.27 1.27)
+			)
 		)
 	)

Commit message: UGR Screen Code TEST
Parts:
- removed R1_BOOT1: 100k, Resistor_SMD:R_0603_1608Metric_Pad0.98x0.95mm_HandSolder, symbol Device:R
- added R1_BOOT0, R1_NRST1: 10k, Resistor_SMD:R_0603_1608Metric_Pad0.98x0.95mm_HandSolder, symbol Device:R
Connections:
- net +3V3: now also R1_NRST1.2
- net GND: now also R1_BOOT0.2
- net NRST: now also R1_NRST1.1
- net at S1.2, U2.94 (BOOT0): now also R1_BOOT0.1
- no-connect marks 54 -> 55
Other:
- moved on the sheet: C_NRST1

Commit message: Stuff
Parts:
- added D2, D3: LED, Connector_PinHeader_2.54mm:PinHeader_1x02_P2.54mm_Vertical, symbol Device:LED
- added R_LED1, R_LED2: 510, Resistor_SMD:R_0603_1608Metric_Pad0.98x0.95mm_HandSolder, symbol Device:R_Small
Connections:
- net +3V3: now also D2.1 (K)
- net +5V: now also D3.1 (K)
- net GND: now also R_LED1.2, R_LED2.2
- new net: D3.2 (A), R_LED2.1
- new net: D2.2 (A), R_LED1.1
Other:
- note added: "CAN TRANSCIEVER"
- note added: "MAIN MCU"
- note added: "POWER LEDs"
- note added: "POWER RAILS"
- moved on the sheet: ABM3-8.000MHZ-10-1-U-T1, C10_U1, C12_U1, C14_U1, C16_U1, C18_U1, C1_CAP1, C1_OSC1, C1_VDD1, C20_U4, C2_CAP1, C2_OSC1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
