File: UGR/New_Screen_26/UGR_Driver_Screen_26_PCB/UGR_Driver_Screen_26.kicad_pcb (KiCad board)
At the start: 2 copper layers, 133.5 x 84 mm, 59 parts, among them J2 USB_B_Micro, J3 Conn_02x20_Socket, J4 Conn_01x06, U1 TPS562200, U2 STM32F767VGTx, U3 SI2347DS-T1-GE3, U4 MCP2562-E-MF, U5 SI2347DS-T1-GE3, U6 SI2347DS-T1-GE3, U7 SI2347DS-T1-GE3, U8 SI2347DS-T1-GE3, U9 SI2347DS-T1-GE3

Commit message: UGR Screen Code TEST
Parts:
- removed R1_BOOT1: 100k, Resistor_SMD:R_0603_1608Metric_Pad0.98x0.95mm_HandSolder
- added R1_BOOT0: 10k, Resistor_SMD:R_0603_1608Metric_Pad0.98x0.95mm_HandSolder, F.Cu at (144.0, 133.5)
- added R1_NRST1: 10k, Resistor_SMD:R_0603_1608Metric_Pad0.98x0.95mm_HandSolder, F.Cu at (132.2, 141.3)
Connections:
- S1 pad 1: Net-(R1_BOOT1-Pad1) -> unconnected-(S1-Pad1)
Routing:
- net Net-(U2-BOOT0): track 39.1 -> 44.1 mm
- net Net-(R1_BOOT1-Pad1): track 3.14 -> 0.00 mm
- net +3V3: track 483.2 -> 485.0 mm
Other:
- board text added: "Boot- Loader"
- board text added: "NRST"
- board text added: "Normal Boot"
- board text removed: "RST"

Commit message: Stuff
Parts:
- added D2_3V3: LED, Connector_PinHeader_2.54mm:PinHeader_1x02_P2.54mm_Vertical, F.Cu at (83.0, 127.5)
- added D3_5V: LED, Connector_PinHeader_2.54mm:PinHeader_1x02_P2.54mm_Vertical, F.Cu at (82.7, 114.5)
- added R_LED1: 510, Resistor_SMD:R_0603_1608Metric_Pad0.98x0.95mm_HandSolder, F.Cu at (83.0, 133.9)
- added R_LED2: 510, Resistor_SMD:R_0603_1608Metric_Pad0.98x0.95mm_HandSolder, F.Cu at (82.6, 121.5)
Routing:
- net +3V3: track 485.0 -> 507.3 mm, vias 12 -> 13
- net +5V: track 132.7 -> 137.5 mm
- net Net-(D3-A): track 0.00 -> 3.71 mm
- net Net-(D2-A): track 0.00 -> 2.99 mm
Other:
- board text added: "V1"

Commit message: Screen V1 REV 7
Parts:
- moved REF** 1.59 mm to (83.0, 140.8)
- moved REF** 1.59 mm to (210.5, 140.8)
- moved REF** 1.26 mm to (210.5, 62.8)
- moved REF** 1.26 mm to (83.0, 62.8)
Routing:
- net GND: vias 33 -> 42
Other:
- board text added: "+"
Changed lines of the file:
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@@
 	(footprint "MountingHole:MountingHole_3.2mm_M3"
 		(layer "F.Cu")
-		(at 82 142)
+		(at 83 140.76)
 		(descr "Mounting Hole 3.2mm, M3, no annular, generated by kicad-footprint-generator mountinghole.py")
 		(tags "mountinghole M3")
 		(property "Reference" "REF**"
-			(at 0 -4.15 0)
+			(at 5.2 1.54 0)
 			(layer "F.SilkS")
 			(effects
@@
 	(footprint "MountingHole:MountingHole_3.2mm_M3"
 		(layer "F.Cu")
-		(at 211.5 62)
+		(at 210.5 62.76)
 		(descr "Mounting Hole 3.2mm, M3, no annular, generated by kicad-footprint-generator mountinghole.py")
 		(tags "mountinghole M3")
 		(property "Reference" "REF**"
-			(at 0 -4.15 0)
+			(at 0 4.34 0)
 			(layer "F.SilkS")
 			(effects
@@
 	(footprint "MountingHole:MountingHole_3.2mm_M3"
 		(layer "F.Cu")
-		(at 82 62)
+		(at 83 62.76)
 		(descr "Mounting Hole 3.2mm, M3, no annular, generated by kicad-footprint-generator mountinghole.py")
 		(tags "mountinghole M3")
 		(property "Reference" "REF**"
-			(at 0 -4.15 0)
+			(at 0 4.34 0)
 			(layer "F.SilkS")
 			(effects
@@
 		(tags "SI2347DS-T1-GE3 ")
 		(property "Reference" "U3"
-			(at 0 0 270)
+			(at 2.5 0 0)
 			(unlocked yes)
 			(layer "F.SilkS")
@@
 	(footprint "MountingHole:MountingHole_3.2mm_M3"
 		(layer "F.Cu")
-		(at 211.5 142)
+		(at 210.5 140.76)
 		(descr "Mounting Hole 3.2mm, M3, no annular, generated by kicad-footprint-generator mountinghole.py")
 		(tags "mountinghole M3")
@@
 	)
 	(gr_rect
-		(start 80 60)
-		(end 213.5 144)
+		(start 80 59.76)
+		(end 213.5 143.76)
 		(stroke
 			(width 0.2)
@@
 	)
 	(gr_text "3V3\n"
-		(at 114.3 142.8 0)
+		(at 114.2 142.7 0)
 		(layer "F.SilkS")
 		(effects
@@
 	)
 	(gr_text "CLK\n"
-		(at 117.5 142.8 0)
+		(at 117.4 142.7 0)
 		(layer "F.SilkS")
 		(effects
@@
 	)
 	(gr_text "5V"
-		(at 111.5 142.8 0)
+		(at 111.4 142.7 0)
 		(layer "F.SilkS")
 		(effects
@@
 		)
 	)
+	(gr_text "+\n"
+		(at 84.2 126.2 0)
+		(layer "F.SilkS")
+		(effects
+			(font
+				(size 1 1)
+				(thickness 0.15)
+			)
+		)
+	)
 	(gr_text "NRST"
-		(at 123 142.8 0)
+		(at 122.9 142.7 0)
+		(layer "F.SilkS")
+		(effects
+			(font
+				(size 1 1)
+				(thickness 0.15)
+			)
+		)
+	)
+	(gr_text "+\n"
+		(at 84 113.2 0)
 		(layer "F.SilkS")
 		(effects
@@
 	)
 	(gr_text "V1\n"
-		(at 205.4 142.5 0)
+		(at 204.8 142.1 0)
 		(layer "F.SilkS")
 		(effects
@@
 	)
 	(gr_text "IO"
-		(at 120 142.8 0)
+		(at 119.9 142.7 0)
 		(layer "F.SilkS")
 		(effects
@@
 	)
 	(gr_text "Designed by Daniel Borkovec\n"
-		(at 185.4 142.3 0)
+		(at 185.7 142 0)
 		(layer "F.SilkS")
 		(effects
@@
 	)
 	(via
+		(at 173.3 88.2)
+		(size 0.6)
+		(drill 0.3)
+		(layers "F.Cu" "B.Cu")
+		(free yes)
+		(net 1)
+	)
+	(via
 		(at 199.4 130.4)
 		(size 0.6)
@@
 	)
 	(via
+		(at 168.7 93)
+		(size 0.6)
+		(drill 0.3)
+		(layers "F.Cu" "B.Cu")
+		(free yes)
+		(net 1)
+	)
+	(via
 		(at 192.7 107.2)
 		(size 0.6)
@@
 	)
 	(via
+		(at 179 102.6)
+		(size 0.6)
+		(drill 0.3)
+		(layers "F.Cu" "B.Cu")
+		(free yes)
+		(net 1)
+	)
+	(via
 		(at 171.7 113.5)
 		(size 0.6)
@@
 	)
 	(via
+		(at 171 85.7)
+		(size 0.6)
+		(drill 0.3)
+		(layers "F.Cu" "B.Cu")
+		(free yes)
+		(net 1)
+	)
+	(via
 		(at 192.7 99.332191)
 		(size 0.6)
@@
 	)
 	(via
+		(at 176.5 100.2)
+		(size 0.6)
+		(drill 0.3)
+		(layers "F.Cu" "B.Cu")
+		(free yes)
+		(net 1)
+	)
+	(via
 		(at 89.8 114.2)
 		(size 0.6)
@@
 	)
 	(via
+		(at 166 90)
+		(size 0.6)
+		(drill 0.3)
+		(layers "F.Cu" "B.Cu")
+		(free yes)
+		(net 1)
+	)
+	(via
 		(at 88.1 128.8)
 		(size 0.6)
@@
 	)
 	(via
+		(at 159.2 96.7)
+		(size 0.6)
+		(drill 0.3)
+		(layers "F.Cu" "B.Cu")
+		(free yes)
+		(net 1)
+	)
+	(via
 		(at 205.4 89.1)
 		(size 0.6)
@@
 	)
 	(via
+		(at 157.2 98.4)
+		(size 0.6)
+		(drill 0.3)
+		(layers "F.Cu" "B.Cu")
+		(free yes)
+		(net 1)
+	)
+	(via
+		(at 192.1 89.4)
+		(size 0.6)
+		(drill 0.3)
+		(layers "F.Cu" "B.Cu")
+		(free yes)
+		(net 1)
+	)
+	(via
 		(at 178.2 107.2)
 		(size 0.6)
@@
 	)
 	(segment
-		(start 179.5 114)
-		(end 180.7 114)
-		(width 0.2)
-		(layer "F.Cu")
-		(net 31)
-	)
-	(segment
 		(start 182.624265 112.075735)
 		(end 182.899 111.801)
@@
 	)
 	(segment
-		(start 212.899 86.879)
-		(end 211.27 85.25)
+		(start 179.5 114)
+		(end 180.7 114)
 		(width 0.2)
 		(layer "F.Cu")
@@
 	)
 	(segment
-		(start 211.74676 111.801)
-		(end 212.899 110.64876)
+		(start 212.899 86.879)
+		(end 211.27 85.25)
 		(width 0.2)
 		(layer "F.Cu")
@@
 		(width 0.2)
 		(layer "F.Cu")
+		(net 31)
+	)
+	(segment
+		(start 211.74676 111.801)
+		(end 212.899 110.64876)
+		(width 0.2)
+		(layer "F.Cu")
